File: LC_Meter_v3.kicad_pro.kicad_sch (KiCad schematic)
At the start: 38 parts, among them J1 TEST, J2 Conn_DC-IN, J3 DC_SEL, J4 Conn_i2c LCD, J5 Conn_i2c LCD2, P2 COM, SW1 SW_DPDT_x2, SW2 SW_DIP_x02, SW3 RESET, U1 74HCU04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

Commit message: Advanced design V1
Parts:
- removed J5: Conn_i2c LCD2, Connector_PinHeader_2.54mm:PinHeader_1x04_P2.54mm_Vertical, symbol Connector_Generic:Conn_01x04
- removed SW2: SW_DIP_x02, Button_Switch_THT:SW_NKK_G1xJP, symbol Switch:SW_DIP_x02
- added H10, H11, H12, H5, H6, H7, H8, H9: MountingHole3.2, MountingHole:MountingHole_3.2mm_M3, symbol Mechanical:MountingHole
- added J5: ICSP, Connector_PinHeader_2.54mm:PinHeader_2x03_P2.54mm_Vertical, symbol Connector_Generic:Conn_02x03_Counter_Clockwise
- added R7: 10k, Resistor_THT:R_Axial_DIN0204_L3.6mm_D1.6mm_P2.54mm_Vertical, symbol Device:R
- added SW2: SW_DPDT_x2, Button_Switch_THT:SW_NKK_G1xJP, symbol Switch:SW_DPDT_x2
- C1, C6: footprint Capacitor_THT:C_Disc_D5.0mm_W2.5mm_P5.00mm -> Capacitor_THT:C_Disc_D3.0mm_W2.0mm_P2.50mm
- C2: footprint Capacitor_SMD:C_0805_2012Metric_Pad1.18x1.45mm_HandSolder -> Capacitor_THT:C_Disc_D3.0mm_W2.0mm_P2.50mm
- C9: footprint Capacitor_THT:C_Disc_D7.5mm_W2.5mm_P5.00mm -> Capacitor_THT:C_Disc_D3.0mm_W2.0mm_P2.50mm
Connections:
- net +5V: now also J5.6 (Pin_6), R7.2
- net 11(**/MOSI): now also J5.5 (Pin_5)
- net 12(MISO): now also J5.1 (Pin_1)
- net 13(SCK): now also J5.2 (Pin_2)
- net 6(**): now also R7.1, SW2.1 (A)
- net GND: now also J5.4 (Pin_4), SW2.2 (B), SW2.5 (B)
- net Reset: now also J5.3 (Pin_3)
- net at C3.1: now also SW2.4 (A)
Other:
- moved on the sheet: C3, C8, H1, H2, H3, H4, P2, Y1
