File: LC_Meter_v3.kicad_pro.kicad_pcb (KiCad board)
At the start: 2 copper layers, 50.2 x 50 mm, 38 parts, among them J1 TEST, J2 Conn_DC-IN, J3 DC_SEL, J4 Conn_i2c LCD, J5 Conn_i2c LCD2, P1 COM, SW1 SW_DPDT_x2, SW2 SW_DIP_x02, SW3 RESET, U1 74HCU04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

Commit message: Advanced design V1
Parts:
- added H10: MountingHole3.2, MountingHole:MountingHole_3.2mm_M3, F.Cu at (96.1, 87.6)
- added H11: MountingHole3.2, MountingHole:MountingHole_3.2mm_M3, F.Cu at (89.5, 80.3)
- added H12: MountingHole3.2, MountingHole:MountingHole_3.2mm_M3, F.Cu at (96.1, 80.7)
- added H5: MountingHole3.2, MountingHole:MountingHole_3.2mm_M3, F.Cu at (119.3, 76.2)
- added H6: MountingHole3.2, MountingHole:MountingHole_3.2mm_M3, F.Cu at (126.9, 76.2)
- added H7: MountingHole3.2, MountingHole:MountingHole_3.2mm_M3, F.Cu at (119.3, 68.2)
- added H8: MountingHole3.2, MountingHole:MountingHole_3.2mm_M3, F.Cu at (126.9, 68.2)
- added H9: MountingHole3.2, MountingHole:MountingHole_3.2mm_M3, F.Cu at (89.3, 87.9)
- added R7: 10k, Resistor_THT:R_Axial_DIN0204_L3.6mm_D1.6mm_P2.54mm_Vertical, F.Cu at (108.1, 92.7)
- C1, C6: footprint Capacitor_THT:C_Disc_D5.0mm_W2.5mm_P5.00mm -> Capacitor_THT:C_Disc_D3.0mm_W2.0mm_P2.50mm
- C7: footprint Capacitor_SMD:C_0805_2012Metric_Pad1.18x1.45mm_HandSolder -> Capacitor_THT:C_Disc_D3.0mm_W2.0mm_P2.50mm
- C9: footprint Capacitor_THT:C_Disc_D7.5mm_W2.5mm_P5.00mm -> Capacitor_THT:C_Disc_D3.0mm_W2.0mm_P2.50mm
- J5: value Conn_i2c LCD2 -> ICSP; footprint Connector_PinHeader_2.54mm:PinHeader_1x04_P2.54mm_Vertical -> Connector_PinHeader_2.54mm:PinHeader_2x03_P2.54mm_Vertical
- SW2: value SW_DIP_x02 -> SW_DPDT_x2
- moved SW2 91.9 mm to (102.4, 99.7), turned to 90 degrees
- moved J5 64.4 mm to (102.8, 106.6), turned to 90 degrees
- moved H3 64.0 mm to (182.5, 108.7), turned to 90 degrees
- moved R5 60.8 mm to (135.3, 105.4), turned to 90 degrees
- moved C12 57.2 mm to (141.3, 108.8), turned to 90 degrees
- moved C11 54.7 mm to (141.8, 100.9), turned to 90 degrees
- moved C8 54.1 mm to (135.4, 95.4), turned to 90 degrees
- moved J3 52.5 mm to (129.5, 109.1), turned to 90 degrees
- moved R3 52.1 mm to (167.8, 109.7), turned to 0 degrees
- moved C2 50.7 mm to (150.2, 109.1), turned to 180 degrees
- moved C7 50.7 mm to (139.6, 95.5), turned to 90 degrees
- moved C4 50.6 mm to (163.9, 109.9), turned to 180 degrees
- moved C13 50.2 mm to (141.1, 104.7), turned to 90 degrees
- moved SW3 49.4 mm to (173.8, 108.8), turned to 90 degrees
- moved H2 49.2 mm to (118.8, 84.3), turned to 90 degrees
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Connections:
- C3 pad 1: Net-(C3-Pad1) -> Net-(SW2B-A)
- J5 pad 1: +5V -> /12(MISO)
- J5 pad 2: /A5 -> /13(SCK)
- J5 pad 3: /A4 -> /Reset
- SW2 pad 2: Net-(C3-Pad1) -> GND
- SW2 pad 3: GND -> unconnected-(SW2A-C-Pad3)
- SW2 pad 4: GND -> Net-(SW2B-A)
- SW2 pad 5: (no net) -> GND
- SW2 pad 6: (no net) -> unconnected-(SW2B-C-Pad6)

Commit message: Updated pcb file
Parts:
- moved H10 54.1 mm to (126.4, 132.4)
- moved H11 54.1 mm to (119.9, 125.1)
- moved H12 54.1 mm to (126.4, 125.6)
- moved H9 54.1 mm to (119.6, 132.7)
Routing:
- removed copper zone on B.Cu, net GND
Other:
- board size 50.2 x 50 mm -> 50.2 x 4.4 mm
Changed lines of the file:
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@@
   )
   (footprint "MountingHole:MountingHole_3.2mm_M3" (layer "F.Cu")
-    (at 89.271 87.851 90)
+    (at 119.624 132.682 90)
     (descr "Mounting Hole 3.2mm, no annular, M3")
     (tags "mounting hole 3.2mm no annular m3")
@@
   )
   (footprint "MountingHole:MountingHole_3.2mm_M3" (layer "F.Cu")
-    (at 89.516 80.307 90)
+    (at 119.869 125.138 90)
     (descr "Mounting Hole 3.2mm, no annular, M3")
     (tags "mounting hole 3.2mm no annular m3")
@@
   )
   (footprint "MountingHole:MountingHole_3.2mm_M3" (layer "F.Cu")
-    (at 96.069 87.597 90)
+    (at 126.422 132.428 90)
     (descr "Mounting Hole 3.2mm, no annular, M3")
     (tags "mounting hole 3.2mm no annular m3")
@@
   )
   (footprint "MountingHole:MountingHole_3.2mm_M3" (layer "F.Cu")
-    (at 96.069 80.739 90)
+    (at 126.422 125.57 90)
     (descr "Mounting Hole 3.2mm, no annular, M3")
     (tags "mounting hole 3.2mm no annular m3")
@@
   (gr_line (start 150.622 112.522) (end 150.622 110.617)
     (stroke (width 0.15) (type solid)) (layer "Dwgs.User"))
-  (gr_line (start 150.876 67.437) (end 143.256 67.437)
-    (stroke (width 0.15) (type solid)) (layer "Dwgs.User"))
-  (gr_line (start 150.876 72.517) (end 150.876 67.437)
-    (stroke (width 0.15) (type solid)) (layer "Dwgs.User"))
   (gr_line (start 143.51 102.997) (end 150.622 102.997)
     (stroke (width 0.15) (type solid)) (layer "Dwgs.User"))
   (gr_line (start 143.51 110.617) (end 143.51 102.997)
     (stroke (width 0.15) (type solid)) (layer "Dwgs.User"))
-  (gr_line (start 143.256 67.437) (end 143.256 72.517)
-    (stroke (width 0.15) (type solid)) (layer "Dwgs.User"))
   (gr_line (start 143.51 112.522) (end 150.622 112.522)
     (stroke (width 0.15) (type solid)) (layer "Dwgs.User"))
   (gr_line (start 143.51 110.617) (end 143.51 112.522)
-    (stroke (width 0.15) (type solid)) (layer "Dwgs.User"))
-  (gr_line (start 143.256 72.517) (end 150.876 72.517)
     (stroke (width 0.15) (type solid)) (layer "Dwgs.User"))
   (gr_line (start 145.542 85.217) (end 149.479 85.217)
@@
   (gr_line (start 145.542 87.757) (end 145.542 85.217)
     (stroke (width 0.15) (type solid)) (layer "Dwgs.User"))
-  (gr_rect (start 115.49 111.6) (end 185.34 81.628)
+  (gr_rect (start 115.49 81.628) (end 185.34 111.6)
     (stroke (width 0.1) (type default)) (fill none) (layer "Eco1.User"))
-  (gr_line (start 115.7 61.6) (end 165.7 61.6)
-    (stroke (width 0.1) (type solid)) (layer "Edge.Cuts"))
   (gr_line (start 115.5 111.6) (end 115.5 111.6)
     (stroke (width 0.1) (type solid)) (layer "Edge.Cuts"))
   (gr_circle (center 163.4 108.8) (end 164.4 110)
-    (stroke (width 0.1) (type solid)) (fill none) (layer "Edge.Cuts"))
-  (gr_line (start 165.7 61.6) (end 165.7 111.6)
-    (stroke (width 0.1) (type solid)) (layer "Edge.Cuts"))
-  (gr_line (start 115.5 111.6) (end 115.7 61.6)
-    (stroke (width 0.1) (type solid)) (layer "Edge.Cuts"))
-  (gr_circle (center 118.6 63.9) (end 119.8 64.9)
     (stroke (width 0.1) (type solid)) (fill none) (layer "Edge.Cuts"))
   (gr_circle (center 118.5 109.1) (end 119.4 110.4)
@@
   (gr_line (start 165.7 111.6) (end 115.5 111.6)
     (stroke (width 0.1) (type solid)) (layer "Edge.Cuts"))
-  (gr_circle (center 163.6 63.8) (end 164.7 64.9)
-    (stroke (width 0.1) (type solid)) (fill none) (layer "Edge.Cuts"))
   (gr_text "nobcha2025\nLC-meter\n" (at 140.626 87.48) (layer "F.Cu")
     (effects (font (size 1.5 1.5) (thickness 0.3)))
@@
     (effects (font (size 1 1) (thickness 0.15)))
   )
-  (dimension (type aligned) (layer "Eco2.User")
-    (pts (xy 165.8 61.5) (xy 165.9 111.5))
-    (height -6.197689)
-    (gr_text "50.0001 mm" (at 173.847673 86.484005 270.1145914) (layer "Eco2.User")
-      (effects (font (size 1.5 1.5) (thickness 0.3)))
-    )
-    (format (prefix "") (suffix "") (units 2) (units_format 1) (precision 4))
-    (style (thickness 0.3) (arrow_length 1.27) (text_position_mode 0) (extension_height 0.58642) (extension_offset 0) keep_text_aligned)
-  )
-  (dimension (type aligned) (layer "Eco2.User")
-    (pts (xy 120.1 109.1) (xy 116.9 109))
-    (height -7.2)
-    (gr_text "3.2016 mm" (at 118.331333 114.447365 -1.789910608) (layer "Eco2.User")
-      (effects (font (size 1.5 1.5) (thickness 0.3)))
-    )
-    (format (prefix "") (suffix "") (units 2) (units_format 1) (precision 4))
-    (style (thickness 0.3) (arrow_length 1.27) (text_position_mode 0) (extension_height 0.58642) (extension_offset 0) keep_text_aligned)
-  )
-  (dimension (type aligned) (layer "Eco2.User")
-    (pts (xy 165.7 111.74157) (xy 115.7 111.9))
-    (height -8.65843)
-    (gr_text "50.0003 mm" (at 140.721732 118.679181 0.1815467994) (layer "Eco2.User")
-      (effects (font (size 1.5 1.5) (thickness 0.3)))
-    )
-    (format (prefix "") (suffix "") (units 2) (units_format 1) (precision 4))
-    (style (thickness 0.3) (arrow_length 1.27) (text_position_mode 0) (extension_height 0.58642) (extension_offset 0) keep_text_aligned)
-  )
-  (dimension (type aligned) (layer "Eco2.User")
-    (pts (xy 163.6 63.9) (xy 163.6 108.8))
-    (height -5.3)
-    (gr_text "44.9000 mm" (at 167.1 86.35 90) (layer "Eco2.User")
-      (effects (font (size 1.5 1.5) (thickness 0.3)))
-    )
-    (format (prefix "") (suffix "") (units 2) (units_format 1) (precision 4))
-    (style (thickness 0.3) (arrow_length 1.27) (text_position_mode 0) (extension_height 0.58642) (extension_offset 0) keep_text_aligned)
-  )
-  (dimension (type aligned) (layer "Eco2.User")
-    (pts (xy 118.7 63.9) (xy 163.6 63.9))
-    (height -4.5)
-    (gr_text "44.9000 mm" (at 141.15 57.6) (layer "Eco2.User")
-      (effects (font (size 1.5 1.5) (thickness 0.3)))
-    )
-    (format (prefix "") (suffix "") (units 2) (units_format 1) (precision 4))
-    (style (thickness 0.3) (arrow_length 1.27) (text_position_mode 0) (extension_height 0.58642) (extension_offset 0) keep_text_aligned)
-  )
-  (dimension (type aligned) (layer "Eco2.User")
-    (pts (xy 163.4 108.9) (xy 118.5 109.1))
-    (height -5.401727)
-    (gr_text "44.9004 mm" (at 140.966043 112.601691 0.2552133656) (layer "Eco2.User")
-      (effects (font (size 1.5 1.5) (thickness 0.3)))
-    )
-    (format (prefix "") (suffix "") (units 2) (units_format 1) (precision 4))
-    (style (thickness 0.3) (arrow_length 1.27) (text_position_mode 0) (extension_height 0.58642) (extension_offset 0) keep_text_aligned)
-  )
-  (zone (net 4) (net_name "GND") (layer "B.Cu") (hatch edge 0.508)
-    (connect_pads (clearance 0.508))
-    (min_thickness 0.254) (filled_areas_thickness no)
-    (fill yes (thermal_gap 0.508) (thermal_bridge_width 0.508))
-    (polygon
-      (pts
-        (xy 165 110.6)
-        (xy 116.5 110.6)
-        (xy 116.5 62.1)
-        (xy 165 62.1)
-      )
-    )
-  )
 )
